Commit message: version final avec quelques bug

File: circuit/src/urdf/include/common_macros.urdf.xacro (robot description, xacro)
@@ -4,4 +4,5 @@
   <xacro:property name="package_name" value="${package_name}" scope="global"/>
 </xacro:macro>
+<!-- <xacro:include filename="$(find circuit)/src/urdf/materials.xacro" /> -->
 <!-- ===================== Wheel xacro =========================================
   Xacro to create a wheel link and the respective joint. For more detail information and usage, see:
@@ -16,5 +17,5 @@
 -->
   <xacro:macro name="wheel"
-               params="prefix reflect wheel_props base_props mesh:='' ">
+               params="prefix reflect wheel_props wheel_color base_props mesh:='' ">
   <xacro:property name="pos_x_joint"
      value="${(base_props['base']['x_size']/2) - wheel_props['wheel']['x_offset']}"/>
@@ -37,5 +38,4 @@
          <cylinder radius="${wheel_props['wheel']['radius']}" length="${wheel_props['wheel']['length']}"/>
         </geometry>
-        <material name="red"/>
       </visual>
     </xacro:if>
@@ -51,4 +51,7 @@
       </xacro:cylinder_inertia>
     </link>
+    <gazebo reference="${prefix}_wheel">
+    <material>Gazebo/${wheel_color}</material>
+    </gazebo>
     <joint name="${prefix}_wheel_joint" type="continuous">
       <axis xyz="0 1 0" rpy="0 0 0" />
@@ -69,5 +72,5 @@
   </xacro:macro>
    <xacro:macro name="camera"
-               params="cam_height cam_rot_y">
+               params="robot_index cam_height cam_rot_y">
   <link name="camera_link">
     <collision>
@@ -82,7 +85,4 @@
     <box size="0.1 0.1 0.1"/>
       </geometry>
-      <material name="Red">
-         <color rgba="1.0 0.0 0.0 1.0"/>
-        </material>
     </visual>
     <inertial>
@@ -123,5 +123,5 @@
         <alwaysOn>true</alwaysOn>
         <updateRate>0.0</updateRate>
-        <cameraName>rrbot/camera1</cameraName>
+        <cameraName>robot_${robot_index}/camera1</cameraName>
         <imageTopicName>image_raw</imageTopicName>
         <cameraInfoTopicName>camera_info</cameraInfoTopicName>
@@ -151,7 +151,5 @@
     <box size="0.05 0.05 0.05"/>
       </geometry>
-       <material name="Cyan">
-         <color rgba="0 1.0 1.0 1.0"/>
-        </material>
+       <!-- <material>Gazebo/Red</material> -->
     </visual>
     <inertial>
@@ -196,5 +194,5 @@
          <alwaysOn>true</alwaysOn>
          <updateRate>50</updateRate>
-         <topicName>sensor_${robot_index}/${prefix}_ir_front</topicName>
+         <topicName>robot_${robot_index}/sensor_${prefix}_ir</topicName>
          <frameName>base_ir_front</frameName>
          <radiation>INFRARED</radiation>
@@ -203,4 +201,7 @@
    </sensor>
    </gazebo>
+<!-- <gazebo reference="${prefix}_sensor_link">
+    <material>Gazebo/Red</material>
+  </gazebo> -->
 </xacro:macro>
 <!-- ======================================================================= -->
@@ -226,5 +227,5 @@
             </geometry>
             <!-- xacro:insert_block name="material_silver" / TODO use this block? -->
-            <material name="silver"/>
+            <!-- <material>Gazebo/Red</material> -->
         </visual>
       </xacro:if>
@@ -235,5 +236,5 @@
             <box size="${wheel_props['base']['size']['x']} ${wheel_props['base']['size']['y']} ${wheel_props['base']['size']['z']}" />
           </geometry>
-          <material name="red"/>
+          <!-- <material>Gazebo/Red</material> -->
         </visual>
       </xacro:if>
@@ -254,5 +255,5 @@
     </joint>
     <gazebo reference="${prefix}_caster_base_link">
-      <material>Gazebo/Grey</material>
+      <!-- <material>Gazebo/Red</material> -->
     </gazebo>
     <!-- caster hub -->
@@ -273,5 +274,5 @@
           </geometry>
           <!-- xacro:insert_block name="material_silver" / TODO use this block? -->
-          <material name="silver"/>
+          <!-- <material>Gazebo/Red</material> -->
         </visual>
       </xacro:if>
@@ -282,5 +283,5 @@
             <box size="${wheel_props['hub']['size']['x']} ${wheel_props['hub']['size']['y']} ${wheel_props['hub']['size']['z']}" />
           </geometry>
-          <material name="red"/>
+          <!-- <material>Gazebo/Red</material> -->
         </visual>
       </xacro:if>
@@ -301,5 +302,5 @@
     </joint>
     <gazebo reference="${prefix}_caster_rotation_link">
-      <material>Gazebo/Grey</material>
+      <!-- <material>Gazebo/Red</material> -->
     </gazebo>
     <!-- caster wheel -->
@@ -316,6 +317,6 @@
             <mesh filename="package://${package_name}/meshes/${robot_name}/${wheel_props['wheel']['mesh']}" />
           </geometry>
-          <!-- TODO use this?: xacro:insert_block name="material_dark_grey" /-->
-          <material name="material_dark_grey"/>
+          <!-- TODO use this?: xacro:insert_block name="material_dark_red" /-->
+          <!-- <material>Gazebo/Red</material> -->
         </visual>
       </xacro:if>
@@ -326,5 +327,8 @@
             <cylinder length="${wheel_props['wheel']['length']}" radius="${wheel_props['wheel']['radius']}" />
           </geometry>
-          <material name="red"/>
+          <material name="Cyan">
+         <color rgba="0 1.0 1.0 1.0"/>
+       </material>
+          <!-- <material>Gazebo/Red</material> -->
         </visual>
       </xacro:if>
@@ -344,5 +348,5 @@
     </joint>
     <gazebo reference="${prefix}_caster_wheel_link">
-      <material>Gazebo/DarkGrey</material>
+      <!-- <material>Gazebo/Red</material> -->
     </gazebo>
   </xacro:macro>
@@ -365,9 +369,9 @@
     </xacro:box_inertia>
       <visual>
-        <origin xyz="0 0 0.1" rpy="0 0 1.57"/>
+        <origin xyz="0.03 0 0.1" rpy="0 0 1.57"/>
         <geometry>
-          <mesh filename="package://circuit/src/urdf/car_blender.dae" scale="0.2 0.2 0.2"/>
-        </geometry>
-        <material name="white" />
+          <mesh filename="package://circuit/src/urdf/meshes/car_blender.dae" scale="0.19 0.2 0.2"/>
+        </geometry>
+        <!-- <material>Gazebo/Red</material> -->
       </visual>
     <collision>
@@ -461,12 +465,12 @@
   RVIZ material RGBA definition.
 -->
-  <material name="blue">
+  <!-- <material name="blue">
     <color rgba="0 0 0.8 1"/>
   </material>
   <material name="black">
-    <color rgba="0 0 0 1"/>
+    <color rgba="0 0 0 1.0"/>
   </material>
   <material name="white">
-    <color rgba="1 1 1 1"/>
+    <color rgba="1.0 1.0 1.0 1.0"/>
   </material>
   <material name="red">
@@ -476,7 +480,7 @@
     <color rgba="0.79 0.82 0.93 1"/>
   </material>
-  <material name="material_dark_grey">
+  <material name="material_dark_red">
     <color rgba="0.3 0.3 0.3 1"/>
-  </material>
+  </material> -->
 <!-- ========================================================================-->
 </robot>

File: circuit/src/urdf/mobile_robot.urdf.xacro (robot description, xacro)
@@ -4,4 +4,5 @@
   <xacro:property name="robot_name" value="mobile_robot"/>
   <xacro:include filename="$(find ${package_name})/src/urdf/include/common_macros.urdf.xacro" />
+  <!-- <xacro:include filename="$(find ${package_name})/src/urdf/materials.xacro" /> -->
   <!-- <xacro:set_package_name /> -->
   <xacro:property name="back_wheel_yaml" value="$(find ${package_name})/src/config/${robot_name}/back_wheel.yaml" />
@@ -18,18 +19,25 @@
   <xacro:wheel prefix="back_right" reflect="-1"
                       wheel_props="${back_wheel_props}"
-                      base_props="${base_props}">
+                      wheel_color="$(arg wheel_color)"
+                      base_props="${base_props}"
+                      >
   </xacro:wheel>
   <xacro:wheel prefix="back_left" reflect="1"
                       wheel_props="${back_wheel_props}"
-                      base_props="${base_props}">
+                      wheel_color="$(arg wheel_color)"
+                      base_props="${base_props}"
+                      >
   </xacro:wheel>
-  <!-- Front Wheels -->
   <xacro:wheel prefix="front_right" reflect="-1"
                       wheel_props="${front_wheel_props}"
-                      base_props="${base_props}">
+                      wheel_color="$(arg wheel_color)"
+                      base_props="${base_props}"
+                      >
   </xacro:wheel>
   <xacro:wheel prefix="front_left" reflect="1"
                       wheel_props="${front_wheel_props}"
-                      base_props="${base_props}">
+                      wheel_color="$(arg wheel_color)"
+                      base_props="${base_props}"
+                      >
   </xacro:wheel>
  <xacro:sensor prefix="left" robot_index="$(arg robot_index)" sensor_x="0" sensor_y="-0.2" sensor_rotate="-1.07"/>
@@ -38,6 +46,6 @@
 <!--  <xacro:sensor prefix="right" sensor_y="-0.5" sensor_rotate="3.1415"/>
 -->
-  <xacro:camera cam_height="0.2" cam_rot_y="0.1"/>
-        <gazebo>
+<xacro:camera robot_index="$(arg robot_index)" cam_height="0.2" cam_rot_y="0.1"/>
+<gazebo>
   <plugin name="skid_steer_drive_controller" filename="libgazebo_ros_skid_steer_drive.so">
     <updateRate>100.0</updateRate>
@@ -47,5 +55,5 @@
     <leftRearJoint>back_left_wheel_joint</leftRearJoint>
     <rightRearJoint>back_right_wheel_joint</rightRearJoint>
-    <wheelSeparation>0.4</wheelSeparation>
+    <wheelSeparation>2</wheelSeparation>
     <wheelDiameter>0.2</wheelDiameter>
     <robotBaseFrame>base_link</robotBaseFrame>
@@ -55,5 +63,4 @@
   </plugin>
 </gazebo>
-<!--
   <gazebo reference="sensor_link">
     <sensor type="camera" name="camera1">
@@ -61,5 +68,4 @@
       </plugin>
     </sensor>
-  </gazebo>-->
-  <!-- <xacro:include filename="$(find mobile_description)/urdf/mobile_robot_gazebo_plugins.xacro"/>  -->
+  </gazebo>
 </robot>

File: circuit/src/urdf/race_track.urdf.xacro (robot description, xacro)
@@ -1,10 +1,13 @@
 <?xml version="1.0"?>
 <robot xmlns:xacro="http://www.ros.org/wiki/xacro" name="race_track">
-<link name="race_track">
+<!-- <xacro:include filename="$(find circuit)/src/urdf/race_track.gazebo" /> -->
+<xacro:include filename="$(find circuit)/src/urdf/materials.xacro" />
+<!-- <xacro:property name="race_track_yaml" value="$(find ${package_name})/src/config/race_track/race_track.yaml" />
+<xacro:property name="race_track_props" value="${load_yaml(race_track_yaml)}"/> -->
+<link name="race_track_link">
     <collision>
       <origin xyz="0 0 0" rpy="0 0 0"/>
       <geometry>
       <mesh filename="package://circuit/src/urdf/meshes/track_map.stl" scale="1 1 1"/>
-        <!-- <box size="1 1 1"/> -->
       </geometry>
     </collision>
@@ -12,8 +15,8 @@
       <origin xyz="0 0 0" rpy="0 0 0"/>
       <geometry>
-      <mesh filename="package://circuit/src/urdf/meshes/track_map.stl" scale="1 1 1"/>
+      <mesh filename="package://circuit/src/urdf/meshes/circuit_visual.dae" scale="1 1 1">
+      </mesh>
         <!-- <box size="1 1 1"/> -->
       </geometry>
-      <material name="orange"/>
     </visual>
     <inertial>
@@ -26,8 +29,161 @@
     </inertial>
 </link>
-<link name="world"/>
+<link name="world">
+<inertial>
+      <origin xyz="0 0 0" rpy="0 0 0"/>
+      <mass value="1"/>
+      <inertia
+        ixx="1.0" ixy="0.0" ixz="0.0"
+        iyy="1.0" iyz="0.0"
+        izz="1.0"/>
+    </inertial>
+  </link>
   <joint name="fixed" type="fixed">
     <parent link="world"/>
-    <child link="race_track"/>
+    <child link="race_track_link"/>
   </joint>
+  <!-- <link name="door">
+    <origin xyz="0 0 2" rpy="0 0 0"/>
+    <collision>
+      <origin xyz="0 0 1" rpy="0 0 0"/>
+      <geometry>
+    <box size="1 0.5 0.5"/>
+      </geometry>
+    </collision>
+    <visual>
+      <origin xyz="0 0 1" rpy="0 0 0"/>
+      <geometry>
+    <box size="1 0.5 0.5"/>
+      </geometry>
+      <material name="Red">
+         <color rgba="1.0 0.0 0.0 1.0"/>
+        </material>
+    </visual>
+    <inertial>
+      <mass value="1e-5" />
+      <origin xyz="0 0 1" rpy="0 0 0"/>
+      <inertia ixx="1e-6" ixy="0" ixz="0" iyy="1e-6" iyz="0" izz="1e-6" />
+    </inertial>
+  </link>
+    <joint name="door_joint" type="continuous">
+      <axis xyz="0 0 1" rpy="0 0 0" />
+      <parent link="race_track_link"/>
+      <child link="door"/>
+      <origin xyz="0 0 0" rpy="0 0 0"/>
+      <dynamics damping="0.7"/>
+    </joint> -->
+  <link name="screen_score">
+    <origin xyz="0 0 0" rpy="0 0 0"/>
+    <collision>
+      <origin xyz="0 0 0" rpy="0 0 0"/>
+      <geometry>
+    <box size="0.5 0.5 0.1"/>
+      </geometry>
+    </collision>
+    <visual>
+      <origin xyz="0 0 0" rpy="0 0 0"/>
+      <geometry>
+    <box size="0.5 0.5 0.1"/>
+      </geometry>
+      <material name="Red">
+         <color rgba="1.0 0.0 0.0 1.0"/>
+        </material>
+    </visual>
+    <inertial>
+      <mass value="1e-5" />
+      <origin xyz="0 0 0" rpy="0 0 0"/>
+      <inertia ixx="1e-6" ixy="0" ixz="0" iyy="1e-6" iyz="0" izz="1e-6" />
+    </inertial>
+  </link>
+    <joint name="screen_joint" type="fixed">
+      <parent link="race_track_link"/>
+      <child link="screen_score"/>
+      <origin xyz="2 1.8 1" rpy="1.57 0 -1.57"/>
+    </joint>
+  <!-- <transmission name="tran2">
+    <type>transmission_interface/SimpleTransmission</type>
+    <joint name="door_joint">
+      <hardwareInterface>hardware_interface/EffortJointInterface</hardwareInterface>
+    </joint>
+    <actuator name="motor2">
+      <hardwareInterface>hardware_interface/EffortJointInterface</hardwareInterface>
+      <mechanicalReduction>1</mechanicalReduction>
+    </actuator>
+  </transmission>  -->
+<gazebo reference="screen_score">
+  <visual>
+    <plugin name="display_video_controller" filename="libgazebo_ros_video.so">
+      <topicName>image_panel</topicName>
+      <height>512</height>
+      <width>512</width>
+    </plugin>
+  </visual>
+</gazebo>
+  <link name="camera_finish">
+  <origin xyz="-2 2.6 0.1" rpy="0 0 -1.57"/>
+    <collision>
+      <origin xyz="0 0 0" rpy="0 0 0"/>
+      <geometry>
+    <box size="0.1 0.1 0.1"/>
+      </geometry>
+    </collision>
+    <visual>
+      <origin xyz="0 0 0" rpy="0 0 0"/>
+      <geometry>
+    <box size="0.1 0.1 0.1"/>
+      </geometry>
+      <material name="Red">
+         <color rgba="1.0 0.0 0.0 1.0"/>
+        </material>
+    </visual>
+    <inertial>
+      <mass value="1e-5" />
+      <origin xyz="0 0 0" rpy="0 0 0"/>
+      <inertia ixx="1e-6" ixy="0" ixz="0" iyy="1e-6" iyz="0" izz="1e-6" />
+    </inertial>
+  </link>
+    <joint name="my_joint" type="fixed">
+    <origin xyz="-2 2.6 0.1" rpy="0 0 -1.57"/>
+   <parent link="race_track_link"/>
+   <child link="camera_finish"/>
+   </joint>
+   <gazebo reference="camera_finish">
+    <sensor type="camera" name="camera1">
+      <update_rate>30.0</update_rate>
+      <camera name="head">
+        <horizontal_fov>1.3962634</horizontal_fov>
+        <image>
+          <width>40</width>
+          <height>40</height>
+          <format>R8G8B8</format>
+        </image>
+        <clip>
+          <near>0.02</near>
+          <far>300</far>
+        </clip>
+        <noise>
+          <type>gaussian</type>
+          <!-- Noise is sampled independently per pixel on each frame.
+               That pixel's noise value is added to each of its color
+               channels, which at that point lie in the range [0,1]. -->
+          <mean>0.0</mean>
+          <stddev>0.007</stddev>
+        </noise>
+      </camera>
+      <plugin name="camera_controller" filename="libgazebo_ros_camera.so">
+        <alwaysOn>true</alwaysOn>
+        <updateRate>0.0</updateRate>
+        <cameraName>/race_track/finish_cam</cameraName>
+        <imageTopicName>image_raw</imageTopicName>
+        <cameraInfoTopicName>camera_info</cameraInfoTopicName>
+        <frameName>camera_link</frameName>
+        <hackBaseline>0.07</hackBaseline>
+        <distortionK1>0.0</distortionK1>
+        <distortionK2>0.0</distortionK2>
+        <distortionK3>0.0</distortionK3>
+        <distortionT1>0.0</distortionT1>
+        <distortionT2>0.0</distortionT2>
+      </plugin>
+    </sensor>
+  </gazebo>
 </robot>
